File: board/badge.brd (EAGLE design)
At the start: 145.6 x 94.8 mm, 11 parts, among them X1 SMA-142-0701-851/861

Commit message: schematic mostly done
Parts:
- removed U$5: JTI_ANTENNA-1575AT43A40, Ava:JTI_ANTENNA-1575AT43A40
- removed U$7: RFM22SMD, SparkFun-RF:RFM22-XXX-S2
- added C1, C10, C2, C3, C4, C9: (no value), rcl:C0603
- added C11, C12: 2u2, rcl:C0603
- added C13, C5, C6: 1u, rcl:C0603
- added C7, C8: (no value), rcl:C1210
- added J1: SWD_PTH_SHROUD, dtb:SWD_PTH_SHROUD
- added J2: (no value), dtb:JST-2-TH
- added JP1: FTDI_DEVICE, SparkFun-Connectors:FTDI_DEVICE_SIDE
- added LED1, LED2: (no value), SparkFun-LED:LED-0603
- added R1, R2, R3, R4, R5, R6: (no value), rcl:R0603
- added R7: 1k, rcl:R0603
- added S1, S2, S3: SWITCH-MOMENTARY-2, SparkFun-Electromechanical:TACTILE_SWITCH_TALL
- added U$10: RFM69HW, hoperf:RFM
- added U$11: MCP1640, ukhas:SOT23-6
- added X2: 1503_02, con-lumberg:1503_02
- U$4: value NTX2-VERTICAL -> INDUCTOR; device Ava:NTX2-VERTICAL -> ukhas:INDUCTOR5X5
- moved U$4 48.4 mm to (23.5, 71.0), flipped to the bottom, turned to 0 degrees
- moved U$2 37.3 mm to (46.2, 38.8), turned to 270 degrees
- moved B2 12.7 mm to (32.6, 46.4)
- moved U$3 12.3 mm to (46.1, 64.8), turned to 270 degrees
- moved U$1 12.3 mm to (41.4, 50.6)
- moved U$6 12.3 mm to (31.2, 51.5)
- moved U$8 12.3 mm to (30.8, 34.5)
- moved X1 12.3 mm to (32.2, 13.0)
- moved U$9 10.8 mm to (46.2, 77.0), turned to 29 degrees
Connections:
- removed net +: B2.+1, B2.+2
- removed net -: B2.-1, B2.-2
- removed net 10_GND: U$3.10_GND
- removed net 12_GND: U$3.12_GND
- removed net 1_GND: U$3.1_GND
- removed net 7_VCC_IO: U$3.7_VCC_IO
- removed net 8_VCC: U$3.8_VCC
- removed net GND: U$7.16, U$7.2, U$7.9
- removed net VBAT: U$1.5
- removed net VDD: U$1.7, U$2.16
- removed net VDDA: U$2.5
- removed net VSS: U$1.6, U$2.15
- new net +3V3: C1.1, C10.1, C13.2, C2.1, C3.1, C4.1, C8.1, C9.1, J1.1, LED1.A, R2.2, S2.A2, U$1.5, U$1.7, U$10.VCC, U$11.5, U$2.16, U$2.5, U$3.6_V_BCKP, U$3.7_VCC_IO, U$3.8_VCC, U$8.VCC
- new net 0V: B2.-1, B2.-2, C1.2, C10.2, C11.1, C12.2, C13.1, C2.2, C3.2, C4.2, C7.2, C8.2, C9.2, J1.3, J1.5, J1.9, JP1.P$6, LED2.C, R1.1, R3.1, R4.1, R7.2, U$1.10, U$1.6, U$10.GNDA, U$10.GNDB, U$11.2, U$2.15, U$3.10_GND, U$3.12_GND, U$3.1_GND, U$8.GND, U$8.RFGND, U$9.P$1, U$9.P$3, X1.G@1, X1.G@2, X1.G@3, X1.G@4, X2.2
- new net ADC1: U$2.6, X2.3
- new net CS: U$10.NSS, U$2.10
- new net DIO0: U$10.DIO0, U$2.2
- new net MISO: U$10.MISO, U$2.12
- new net MOSI: U$1.12, U$10.MOSI, U$2.13
- new net N$1: U$3.11_RF_IN, U$9.P$2
- new net N$10: C5.2, U$1.3
- new net N$11: C6.2, U$1.1
- new net N$12: C5.1, U$1.4
- new net N$13: C6.1, U$1.2
- new net N$14: R2.1, R3.2, U$11.4
- new net N$15: U$11.1, U$4.P$2
- new net N$16: C12.1, U$1.14
- new net N$17: LED2.A, R6.1
- new net N$19: R7.1, S3.A2
- new net N$2: U$2.9, U$3.2_TXD1
- new net N$3: LED1.C, R5.2
- new net N$4: U$8.RF, X1.1
- new net N$5: R4.2, U$1.13
- new net N$6: U$10.ANT
- new net N$7: R1.2, S2.B2, U$2.1
- new net N$8: JP1.P$3, U$2.17, U$3.3_RXD1
- new net N$9: JP1.P$2, U$2.18
- new net NRST: J1.10, U$2.4
- new net O_CS: U$1.8, U$2.8
- new net O_RES: U$1.9, U$2.7
- new net SCK: U$1.11, U$10.SCK, U$2.11
- new net SWCLK: J1.4, R6.2, U$2.20
- new net SWDAT: J1.2, R5.1, U$2.19
- new net TX: U$2.14
- new net TX_EN: S3.B2, U$2.3
- new net VIN: B2.+1, B2.+2, C7.1, U$11.3, U$11.6, U$4.P$1
- net VCC: now also C11.2
Other:
- board size 145.6 x 94.8 mm -> 157.3 x 91.3 mm

Commit message: got bored, moved parts around
Parts:
- added SV1: (no value), con-lstb:MA03-1
- moved LED1 204.8 mm to (38.8, 78.8)
- moved R5 204.1 mm to (37.5, 72.8), flipped to the bottom
- moved R6 201.3 mm to (29.0, 73.0), flipped to the bottom
- moved LED2 196.5 mm to (23.5, 78.5)
- moved C13 181.1 mm to (37.2, 51.2), flipped to the bottom, turned to 180 degrees
- moved C12 180.2 mm to (36.2, 54.5), flipped to the bottom, turned to 270 degrees
- moved R4 179.5 mm to (38.2, 54.5), flipped to the bottom, turned to 270 degrees
- moved C11 179.4 mm to (39.2, 57.0), flipped to the bottom
- moved C7 165.7 mm to (25.0, 69.2), flipped to the bottom, turned to 270 degrees
- moved C8 164.1 mm to (17.8, 69.0), flipped to the bottom, turned to 270 degrees
- moved C5 152.6 mm to (38.0, 47.5), flipped to the bottom, turned to 270 degrees
- moved C6 152.6 mm to (38.0, 44.0), flipped to the bottom, turned to 270 degrees
- moved R1 148.5 mm to (41.0, 24.5), flipped to the bottom, turned to 270 degrees
- moved JP1 40.1 mm to (55.2, 59.0), turned to 90 degrees
- moved U$2 1.16 mm to (46.2, 39.9), turned to 180 degrees
Connections:
- net NRST: now also SV1.3
- net SWCLK: now also SV1.2
- net SWDAT: now also SV1.1

Commit message: added mtx2 jumpers
Parts:
- added SJ1, SJ2: (no value), jumper:SJ_2
- moved R1 2.30 mm to (42.5, 26.2)
Connections:
- new net N$18: SJ2.2, U$8.P1
- new net N$20: SJ1.2, U$8.P0
- net +3V3: now also SJ1.1, SJ2.1
- net 0V: now also S1.A2, SJ1.3, SJ2.3
- net NRST: now also S1.B2
- net TX: now also U$8.TXD
- net TX_EN: now also U$8.EN
Changed lines of the file:
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@@
 <layer number="23" name="tOrigins" color="15" fill="1" visible="yes" active="yes"/>
 <layer number="24" name="bOrigins" color="15" fill="1" visible="yes" active="yes"/>
-<layer number="25" name="tNames" color="7" fill="1" visible="yes" active="yes"/>
-<layer number="26" name="bNames" color="7" fill="1" visible="yes" active="yes"/>
-<layer number="27" name="tValues" color="7" fill="1" visible="yes" active="yes"/>
-<layer number="28" name="bValues" color="7" fill="1" visible="yes" active="yes"/>
+<layer number="25" name="tNames" color="7" fill="1" visible="no" active="yes"/>
+<layer number="26" name="bNames" color="7" fill="1" visible="no" active="yes"/>
+<layer number="27" name="tValues" color="7" fill="1" visible="no" active="yes"/>
+<layer number="28" name="bValues" color="7" fill="1" visible="no" active="yes"/>
 <layer number="29" name="tStop" color="7" fill="3" visible="no" active="yes"/>
 <layer number="30" name="bStop" color="7" fill="6" visible="no" active="yes"/>
@@
 <element name="C5" library="rcl" package="C0603" value="1u" x="38" y="47.5" rot="MR270"/>
 <element name="C6" library="rcl" package="C0603" value="1u" x="38" y="44" rot="MR270"/>
-<element name="R1" library="rcl" package="R0603" value="" x="41" y="24.5" rot="MR270"/>
+<element name="R1" library="rcl" package="R0603" value="" x="42.5" y="26.25" rot="MR270"/>
 <element name="R2" library="rcl" package="R0603" value="" x="-95.75" y="-37"/>
 <element name="R3" library="rcl" package="R0603" value="" x="-95.75" y="-40.5"/>
@@
 <attribute name="OC_FARNELL" value="unknown" x="55.25" y="44.5" size="1.778" layer="27" rot="R90" display="off"/>
 </element>
+<element name="SJ1" library="jumper" package="SJ_2" value="" x="40.75" y="23" rot="MR270"/>
+<element name="SJ2" library="jumper" package="SJ_2" value="" x="23.5" y="24.75" rot="MR270"/>
 </elements>
 <signals>
@@
 <contactref element="LED1" pad="A"/>
 <contactref element="S2" pad="A2"/>
+<contactref element="SJ2" pad="1"/>
+<contactref element="SJ1" pad="1"/>
+<wire x1="40.75" y1="24.524" x2="23.5" y2="26.274" width="0" layer="19" extent="1-1"/>
+<wire x1="-96.35" y1="-58" x2="40.75" y2="24.524" width="0" layer="19" extent="1-1"/>
 <wire x1="-96.35" y1="-54.5" x2="-96.35" y2="-58" width="0" layer="19" extent="1-1"/>
 <wire x1="-94.9" y1="-37" x2="-96.35" y2="-54.5" width="0" layer="19" extent="1-1"/>
@@
 <contactref element="U$1" pad="10"/>
 <contactref element="R7" pad="2"/>
+<contactref element="SJ1" pad="3"/>
+<contactref element="SJ2" pad="3"/>
+<contactref element="S1" pad="A2"/>
 <wire x1="-94.65" y1="-58" x2="-100.65" y2="-83.75" width="0" layer="19" extent="1-1"/>
 <wire x1="-94.65" y1="-54.5" x2="-94.65" y2="-58" width="0" layer="19" extent="1-1"/>
@@
 <wire x1="23.9525" y1="45.09875" x2="20.11125" y2="45.09875" width="0" layer="19" extent="16-16"/>
 <wire x1="24.22" y1="29.75" x2="13.27045" y2="37.19759375" width="0" layer="19" extent="16-16"/>
-<wire x1="36.4" y1="51.25" x2="23.9525" y2="45.09875" width="0" layer="19" extent="16-16"/>
-<wire x1="36.25" y1="53.65" x2="36.4" y2="51.25" width="0" layer="19" extent="16-16"/>
-<wire x1="38.25" y1="55.35" x2="36.25" y2="53.65" width="0" layer="19" extent="16-16"/>
+<wire x1="30.25" y1="28.225" x2="24.22" y2="29.75" width="0" layer="19" extent="1-1"/>
+<wire x1="23.5" y1="23.226" x2="24.22" y2="29.75" width="0" layer="19" extent="16-16"/>
+<wire x1="27.8304" y1="15.5654" x2="23.5" y2="23.226" width="0" layer="19" extent="16-16"/>
+<wire x1="27.8304" y1="15.5654" x2="27.8304" y2="15.5654" width="0" layer="19" extent="1-16"/>
+<wire x1="36.6696" y1="15.5654" x2="27.8304" y2="15.5654" width="0" layer="19" extent="1-16"/>
+<wire x1="36.6696" y1="15.5654" x2="36.6696" y2="15.5654" width="0" layer="19" extent="1-16"/>
+<wire x1="40.75" y1="21.476" x2="36.6696" y2="15.5654" width="0" layer="19" extent="1-16"/>
+<wire x1="42.5" y1="27.1" x2="40.75" y2="21.476" width="0" layer="19" extent="16-16"/>
+<wire x1="45.885" y1="29.98" x2="42.5" y2="27.1" width="0" layer="19" extent="16-16"/>
+<wire x1="45.885" y1="31.25" x2="45.885" y2="29.98" width="0" layer="19" extent="1-1"/>
+<wire x1="45.885" y1="33.79" x2="45.885" y2="31.25" width="0" layer="19" extent="1-1"/>
+<wire x1="46.545" y1="37.0222" x2="45.885" y2="33.79" width="0" layer="19" extent="16-16"/>
+<wire x1="40.72" y1="39.25" x2="46.545" y2="37.0222" width="0" layer="19" extent="16-16"/>
+<wire x1="41.4" y1="49.3" x2="40.72" y2="39.25" width="0" layer="19" extent="16-16"/>
+<wire x1="41.4" y1="51.9" x2="41.4" y2="49.3" width="0" layer="19" extent="16-16"/>
+<wire x1="38.25" y1="55.35" x2="41.4" y2="51.9" width="0" layer="19" extent="16-16"/>
 <wire x1="40.1" y1="57" x2="38.25" y2="55.35" width="0" layer="19" extent="16-16"/>
-<wire x1="41.4" y1="51.9" x2="38.25" y2="55.35" width="0" layer="19" extent="16-16"/>
-<wire x1="41.4" y1="49.3" x2="41.4" y2="51.9" width="0" layer="19" extent="16-16"/>
+<wire x1="36.25" y1="53.65" x2="38.25" y2="55.35" width="0" layer="19" extent="16-16"/>
+<wire x1="36.4" y1="51.25" x2="36.25" y2="53.65" width="0" layer="19" extent="16-16"/>
 <wire x1="32.626096875" y1="58.188971875" x2="36.25" y2="53.65" width="0" layer="19" extent="16-16"/>
-<wire x1="40.72" y1="39.25" x2="41.4" y2="49.3" width="0" layer="19" extent="16-16"/>
-<wire x1="46.545" y1="37.0222" x2="40.72" y2="39.25" width="0" layer="19" extent="16-16"/>
-<wire x1="45.885" y1="33.79" x2="46.545" y2="37.0222" width="0" layer="19" extent="16-16"/>
-<wire x1="45.885" y1="31.25" x2="45.885" y2="33.79" width="0" layer="19" extent="1-1"/>
-<wire x1="45.885" y1="29.98" x2="45.885" y2="31.25" width="0" layer="19" extent="1-1"/>
-<wire x1="41" y1="25.35" x2="45.885" y2="29.98" width="0" layer="19" extent="16-16"/>
-<wire x1="36.6696" y1="15.5654" x2="41" y2="25.35" width="0" layer="19" extent="1-16"/>
-<wire x1="36.6696" y1="15.5654" x2="36.6696" y2="15.5654" width="0" layer="19" extent="1-16"/>
-<wire x1="27.8304" y1="15.5654" x2="36.6696" y2="15.5654" width="0" layer="19" extent="1-16"/>
-<wire x1="27.8304" y1="15.5654" x2="27.8304" y2="15.5654" width="0" layer="19" extent="1-16"/>
 <wire x1="50.49" y1="59.85" x2="40.1" y2="57" width="0" layer="19" extent="16-16"/>
 <wire x1="55.25" y1="65.35" x2="50.49" y2="59.85" width="0" layer="19" extent="16-16"/>
@@
 <contactref element="U$2" pad="4"/>
 <contactref element="SV1" pad="3"/>
+<contactref element="S1" pad="B2"/>
 <wire x1="45.245" y1="42.8578" x2="55.25" y2="47.04" width="0" layer="19" extent="16-16"/>
 <wire x1="44.615" y1="33.79" x2="45.245" y2="42.8578" width="0" layer="19" extent="16-16"/>
+<wire x1="25.75" y1="28.225" x2="44.615" y2="33.79" width="0" layer="19" extent="1-1"/>
 </signal>
 <signal name="N$2">
@@
 <contactref element="R1" pad="2"/>
 <contactref element="S2" pad="B2"/>
-<wire x1="41" y1="23.65" x2="43.295" y2="42.8578" width="0" layer="19" extent="16-16"/>
-<wire x1="38.25" y1="20.275" x2="41" y2="23.65" width="0" layer="19" extent="1-16"/>
+<wire x1="42.5" y1="25.4" x2="43.295" y2="42.8578" width="0" layer="19" extent="16-16"/>
+<wire x1="38.25" y1="20.275" x2="42.5" y2="25.4" width="0" layer="19" extent="1-16"/>
 </signal>
 <signal name="N$14">
@@
 <signal name="TX">
 <contactref element="U$2" pad="14"/>
+<contactref element="U$8" pad="TXD"/>
+<wire x1="40.72" y1="33.25" x2="47.195" y2="37.0222" width="0" layer="19" extent="16-16"/>
 </signal>
 <signal name="N$3">
@@
 <contactref element="U$2" pad="3"/>
 <contactref element="S3" pad="B2"/>
+<contactref element="U$8" pad="EN"/>
+<wire x1="40.72" y1="31.25" x2="44.595" y2="42.8578" width="0" layer="19" extent="16-16"/>
 <wire x1="11.25" y1="55.725" x2="44.595" y2="42.8578" width="0" layer="19" extent="1-16"/>
 </signal>
@@
 <wire x1="15.75" y1="55.725" x2="-102.35" y2="-83.75" width="0" layer="19" extent="1-1"/>
 </signal>
+<signal name="N$18">
+<contactref element="U$8" pad="P1"/>
+<contactref element="SJ2" pad="2"/>
+<wire x1="40.72" y1="35.25" x2="23.5" y2="24.75" width="0" layer="19" extent="1-1"/>
+</signal>
+<signal name="N$20">
+<contactref element="SJ1" pad="2"/>
+<contactref element="U$8" pad="P0"/>
+<wire x1="40.72" y1="37.25" x2="40.75" y2="23" width="0" layer="19" extent="1-1"/>
+</signal>
 </signals>
