File: board/badge.brd (EAGLE design)
At the start: 55.6 x 67.5 mm, 50 parts, among them IC1 STM32F030F4, IC2 UBLOX_MAX, IC3 RFM69HW, IC4 MCP1640, J2 20-0096, J3 SWD_PTH_SHROUD, X1 RADIOMETRIX-MTX2, X2 SMA-142-0701-851/861, X3 091OLED

Commit message: some small changes
Routing:
- net 0V: track 191.6 -> 194.3 mm, vias 143 -> 142
Other:
- outline, holes or cut-outs redrawn
Changed lines of the file:
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@@
 <layer number="38" name="bTest" color="7" fill="1" visible="yes" active="yes"/>
 <layer number="39" name="tKeepout" color="4" fill="11" visible="no" active="yes"/>
-<layer number="40" name="bKeepout" color="1" fill="11" visible="yes" active="yes"/>
+<layer number="40" name="bKeepout" color="1" fill="11" visible="no" active="yes"/>
 <layer number="41" name="tRestrict" color="4" fill="10" visible="no" active="yes"/>
 <layer number="42" name="bRestrict" color="1" fill="10" visible="no" active="yes"/>
@@
 <wire x1="8.125" y1="40.5" x2="16.25" y2="28.75" width="0" layer="20"/>
 <wire x1="16.25" y1="28.75" x2="20.25" y2="23" width="0" layer="20"/>
-<wire x1="26.5" y1="13.75" x2="38.25" y2="13.75" width="0" layer="20"/>
+<wire x1="26.5" y1="13.75" x2="38.5" y2="13.75" width="0" layer="20"/>
 <wire x1="57.375" y1="40.75" x2="48.5" y2="28.75" width="0" layer="20"/>
 <text x="48" y="33.5" size="1.016" layer="22" font="vector" ratio="14" rot="SMR90">3.3V only</text>
@@
 <rectangle x1="16.25" y1="28" x2="17.75" y2="31.5" layer="29" rot="R315"/>
 <wire x1="20.25" y1="23" x2="26.5" y2="13.75" width="0" layer="20"/>
-<wire x1="44.5" y1="23" x2="38.25" y2="13.75" width="0" layer="20"/>
+<wire x1="44.5" y1="23" x2="38.5" y2="13.75" width="0" layer="20"/>
 <wire x1="48.5" y1="28.75" x2="44.5" y2="23" width="0" layer="20"/>
 <wire x1="32.625" y1="12.75" x2="32.625" y2="85.375" width="0" layer="51" style="longdash"/>
-<text x="40" y="17.25" size="1.016" layer="21" font="vector" ratio="14" rot="R56">Rev. A May '14</text>
+<text x="40" y="17.25" size="1.016" layer="21" font="vector" ratio="14" rot="R58">Rev. A May '14</text>
 <wire x1="26.9875" y1="78.4225" x2="38.4175" y2="78.4225" width="0" layer="20"/>
 <wire x1="38.4175" y1="78.4225" x2="40.005" y2="76.835" width="0" layer="20" curve="-90"/>
@@
 <wire x1="52.149375" y1="44.846875" x2="52.149375" y2="55.165625" width="0" layer="20"/>
 <wire x1="52.149375" y1="55.165625" x2="53.260625" y2="56.276875" width="0" layer="20" curve="-90"/>
+<wire x1="30.5" y1="40" x2="34.75" y2="40" width="0.4064" layer="22"/>
+<wire x1="35.75" y1="58.25" x2="38.75" y2="58.25" width="0.4064" layer="22"/>
+<wire x1="37.25" y1="56.75" x2="37.25" y2="59.75" width="0.4064" layer="22"/>
+<wire x1="29.5" y1="58.25" x2="26.5" y2="58.25" width="0.4064" layer="22"/>
+<wire x1="28" y1="56.75" x2="28" y2="59.75" width="0.4064" layer="22"/>
 </plain>
 <attributes>
@@
 <wire x1="25.25" y1="24.976" x2="22.024" y2="24.976" width="0.254" layer="16"/>
 <wire x1="40" y1="24.476" x2="34.602096875" y2="24.476" width="0.254" layer="16"/>
-<wire x1="34.602096875" y1="24.476" x2="32.626096875" y2="22.5" width="0.254" layer="16"/>
 <wire x1="28.2054" y1="16.3154" x2="28.2054" y2="19.8304" width="0.3048" layer="1"/>
 <wire x1="31.125" y1="22.75" x2="31.125" y2="27.85" width="0.3048" layer="1"/>
@@
 <via x="19.5" y="35.5" extent="1-16" drill="0.3"/>
 <via x="29.5" y="37.5" extent="1-16" drill="0.3"/>
-<via x="32.75" y="74.5" extent="1-16" drill="0.3"/>
+<wire x1="32.75" y1="74.5" x2="32.75" y2="74.5" width="0" layer="19" extent="1-16"/>
 <via x="37.5" y="73.25" extent="1-16" drill="0.3"/>
 <wire x1="25.5" y1="68.95" x2="25.2" y2="68.95" width="0.4064" layer="16"/>
@@
 <via x="37.5" y="63" extent="1-16" drill="0.3"/>
 <via x="36.25" y="64.25" extent="1-16" drill="0.3"/>
+<wire x1="32.625" y1="19.25" x2="32.625" y2="24.75" width="1.27" layer="16"/>
 </signal>
 <signal name="N$8">
@@
 <via x="47.75" y="44.25" extent="1-16" drill="0.3"/>
 <wire x1="48.34" y1="57.41" x2="49" y2="56.75" width="0.254" layer="16"/>
-<wire x1="49" y1="56.75" x2="49" y2="49" width="0.254" layer="16"/>
-<wire x1="48.25" y1="48.25" x2="48.25" y2="44.75" width="0.254" layer="16"/>
-<wire x1="48.25" y1="44.75" x2="47.75" y2="44.25" width="0.254" layer="16"/>
-<wire x1="49" y1="49" x2="48.25" y2="48.25" width="0.254" layer="16"/>
+<wire x1="49" y1="56.75" x2="49" y2="48.5" width="0.254" layer="16"/>
+<wire x1="48.5" y1="45" x2="47.75" y2="44.25" width="0.254" layer="16"/>
 <wire x1="40.25" y1="44.5" x2="38.75" y2="43" width="0.254" layer="1"/>
 <wire x1="38.75" y1="43" x2="38.75" y2="42.5" width="0.254" layer="1"/>
@@
 <wire x1="42.25" y1="36.75" x2="42.25" y2="41" width="0.254" layer="16"/>
 <wire x1="42.25" y1="41" x2="41.5" y2="41.75" width="0.254" layer="16"/>
+<wire x1="48.5" y1="45" x2="48.5" y2="48" width="0.254" layer="16"/>
+<wire x1="48.5" y1="48" x2="49" y2="48.5" width="0.254" layer="16"/>
 </signal>
 <signal name="N$9">
@@
 <wire x1="49" y1="45.75" x2="49" y2="47.5" width="0.254" layer="1"/>
 <wire x1="49" y1="47.5" x2="49.25" y2="47.75" width="0.254" layer="1"/>
-<wire x1="49.44" y1="47.94" x2="49.44" y2="48.19" width="0.254" layer="16"/>
-<wire x1="49.44" y1="48.19" x2="49.5" y2="48.25" width="0.254" layer="16"/>
-<wire x1="49.5" y1="48.25" x2="49.5" y2="58.54" width="0.254" layer="16"/>
+<wire x1="49.5" y1="48" x2="49.5" y2="58.54" width="0.254" layer="16"/>
 <wire x1="49.5" y1="58.54" x2="49.44" y2="58.6" width="0.254" layer="16"/>
+<wire x1="49.5" y1="48" x2="49.25" y2="47.75" width="0.254" layer="16"/>
 </signal>
 <signal name="N$7">
