File: board/badge.sch (EAGLE design)
At the start: 10 parts, among them X1 SMA-142-0701-851/861

Commit message: schematic mostly done
Parts:
- removed U$5: JTI_ANTENNA-1575AT43A40, Ava:JTI_ANTENNA-1575AT43A40
- removed U$7: RFM22SMD, SparkFun-RF:RFM22SMD
- added C1, C10, C2, C3, C4, C9: (no value), rcl:C-EUC0603
- added C11, C12: 2u2, rcl:C-EUC0603
- added C13, C5, C6: 1u, rcl:C-EUC0603
- added C7, C8: (no value), rcl:C-EUC1210
- added J1: SWD_PTH_SHROUD, dtb:SWD_PTH_SHROUD
- added J2: (no value), dtb:JST_2MM_MALE_TH
- added JP1: FTDI_DEVICE, SparkFun-Connectors:FTDI_DEVICE
- added LED1, LED2: (no value), SparkFun-LED:LED0603
- added R1, R2, R3, R4, R5, R6: (no value), rcl:R-EU_R0603
- added R7: 1k, rcl:R-EU_R0603
- added S1, S2, S3: SWITCH-MOMENTARY-2, SparkFun-Electromechanical:SWITCH-MOMENTARY-2
- added U$10: RFM69HW, hoperf:RFM69HW
- added U$11: MCP1640, ukhas:MCP1640
- added X2: 1503_02, con-lumberg:1503_02
- U$4: value NTX2-VERTICAL -> INDUCTOR; device Ava:NTX2-VERTICAL -> ukhas:INDUCTOR
Connections:
- new net +3V3: C1.1, C10.1, C13.2, C2.1, C3.1, C4.1, C8.1, C9.1, J1.VCC, LED1.A, R2.2, S2.1, U$1.VBAT, U$1.VDD, U$10.VCC, U$11.VOUT, U$2.VDD, U$2.VDDA, U$3.6_V_BCKP, U$3.7_VCC_IO, U$3.8_VCC, U$8.VCC
- new net 0V: B2.-, C1.2, C10.2, C11.1, C12.2, C13.1, C2.2, C3.2, C4.2, C7.2, C8.2, C9.2, J1.GND1, J1.GND2, J1.GNDD, JP1.GND, LED2.C, R1.1, R3.1, R4.1, R7.2, U$1.D/C, U$1.VSS, U$10.GNDA, U$10.GNDB, U$11.GND, U$2.VSS, U$3.10_GND, U$3.12_GND, U$3.1_GND, U$8.0V, U$8.RFGND, U$9.GND, U$9.GND2, X1.2, X2.2
- new net ADC1: U$2.PA0, X2.3
- new net CS: U$10.NSS, U$2.PA4
- new net DIO0: U$10.DIO0, U$2.PF0
- new net MISO: U$10.MISO, U$2.PA6
- new net MOSI: U$1.SDIN, U$10.MOSI, U$2.PA7
- new net N$1: U$3.11_RF_IN, U$9.FEED
- new net N$10: C5.2, U$1.C1P
- new net N$11: C6.2, U$1.C2P
- new net N$12: C5.1, U$1.C1N
- new net N$13: C6.1, U$1.C2N
- new net N$14: R2.1, R3.2, U$11.FB
- new net N$15: U$11.SW, U$4.2
- new net N$16: C12.1, U$1.VCOMH
- new net N$17: LED2.A, R6.1
- new net N$19: R7.1, S3.1
- new net N$2: U$2.PA3, U$3.2_TXD1
- new net N$3: LED1.C, R5.2
- new net N$4: U$8.RFOUT, X1.1
- new net N$5: R4.2, U$1.IREF
- new net N$6: U$10.ANT
- new net N$7: R1.2, S2.2, U$2.BOOT0
- new net N$8: JP1.RXI, U$2.PA9, U$3.3_RXD1
- new net N$9: JP1.TXO, U$2.PA10
- new net NRST: J1.NRST, U$2.NRST
- new net O_CS: U$1.CS, U$2.PA2
- new net O_RES: U$1.RES, U$2.PA1
- new net SCK: U$1.SCLK, U$10.SCK, U$2.PA5
- new net SWCLK: J1.SWCLK, R6.2, U$2.PA14
- new net SWDAT: J1.SWDAT, R5.1, U$2.PA13
- new net TX: U$2.PB1
- new net TX_EN: S3.2, U$2.PF1
- new net VCC: C11.2, U$1.VCC
- new net VIN: B2.+, C7.1, U$11.EN, U$11.VIN, U$4.1
Other:
- note added: "??"
- note added: "check these pins"
- note added: "check with arko >"
- note added: "see rapid 20-0096"
- moved on the sheet: B2, U$1, U$2, X1

Commit message: got bored, moved parts around
Parts:
- added SV1: (no value), con-lstb:MA03-1
Connections:
- net NRST: now also SV1.3
- net SWCLK: now also SV1.2
- net SWDAT: now also SV1.1
Changed lines of the file:
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@@
 <part name="R7" library="rcl" deviceset="R-EU_" device="R0603" value="1k"/>
 <part name="+3V14" library="supply1" deviceset="+3V3" device=""/>
+<part name="SV1" library="con-lstb" deviceset="MA03-1" device=""/>
 </parts>
 <sheets>
@@
 <instance part="R7" gate="G$1" x="-22.86" y="43.18" rot="R180"/>
 <instance part="+3V14" gate="G$1" x="-91.44" y="96.52" rot="R90"/>
+<instance part="SV1" gate="G$1" x="58.42" y="45.72" rot="R180"/>
 </instances>
 <busses>
@@
 <label x="-81.28" y="10.16" size="1.778" layer="95"/>
 </segment>
+<segment>
+<wire x1="35.56" y1="48.26" x2="50.8" y2="48.26" width="0.1524" layer="91"/>
+<label x="40.64" y="48.26" size="1.778" layer="95"/>
+<pinref part="SV1" gate="G$1" pin="1"/>
+</segment>
 </net>
 <net name="SWCLK" class="0">
@@
 <label x="-58.42" y="27.94" size="1.778" layer="95"/>
 </segment>
+<segment>
+<wire x1="35.56" y1="45.72" x2="50.8" y2="45.72" width="0.1524" layer="91"/>
+<label x="40.64" y="45.72" size="1.778" layer="95"/>
+<pinref part="SV1" gate="G$1" pin="2"/>
+</segment>
 </net>
 <net name="NRST" class="0">
@@
 <wire x1="-68.58" y1="101.6" x2="-78.74" y2="101.6" width="0.1524" layer="91"/>
 <label x="-76.2" y="101.6" size="1.778" layer="95"/>
+</segment>
+<segment>
+<wire x1="35.56" y1="43.18" x2="50.8" y2="43.18" width="0.1524" layer="91"/>
+<label x="40.64" y="43.18" size="1.778" layer="95"/>
+<pinref part="SV1" gate="G$1" pin="3"/>
 </segment>
 </net>
@@
 <wire x1="-5.08" y1="43.18" x2="-5.08" y2="33.02" width="0.1524" layer="91"/>
 <label x="-5.08" y="33.02" size="1.778" layer="95"/>
-</segment>
-<segment>
+<junction x="-5.08" y="43.18"/>
+</segment>
+<segment>

Commit message: added mtx2 jumpers
Parts:
- added SJ1, SJ2: (no value), jumper:SJ2W
Connections:
- new net N$18: SJ2.2, U$8.P1
- new net N$20: SJ1.2, U$8.P0
- net +3V3: now also SJ1.1, SJ2.1
- net 0V: now also S1.1, SJ1.3, SJ2.3
- net NRST: now also S1.2
- net TX: now also U$8.TXD
- net TX_EN: now also U$8.EN
Other:
- moved on the sheet: S1
Changed lines of the file:
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@@
 <part name="+3V14" library="supply1" deviceset="+3V3" device=""/>
 <part name="SV1" library="con-lstb" deviceset="MA03-1" device=""/>
+<part name="SJ1" library="jumper" deviceset="SJ2W" device=""/>
+<part name="SJ2" library="jumper" deviceset="SJ2W" device=""/>
+<part name="+3V15" library="supply1" deviceset="+3V3" device=""/>
+<part name="+3V16" library="supply1" deviceset="+3V3" device=""/>
+<part name="GND32" library="supply1" deviceset="0V" device=""/>
+<part name="GND33" library="supply1" deviceset="0V" device=""/>
+<part name="GND34" library="supply1" deviceset="0V" device=""/>
 </parts>
 <sheets>
@@
 <instance part="JP1" gate="G$1" x="55.88" y="66.04"/>
 <instance part="X2" gate="G$1" x="12.7" y="53.34"/>
-<instance part="S1" gate="G$1" x="-99.06" y="104.14"/>
+<instance part="S1" gate="G$1" x="-83.82" y="101.6"/>
 <instance part="S2" gate="G$1" x="-83.82" y="96.52"/>
 <instance part="J1" gate="G$1" x="-12.7" y="129.54"/>
@@
 <instance part="+3V14" gate="G$1" x="-91.44" y="96.52" rot="R90"/>
 <instance part="SV1" gate="G$1" x="58.42" y="45.72" rot="R180"/>
+<instance part="SJ1" gate="G$1" x="251.46" y="58.42"/>
+<instance part="SJ2" gate="G$1" x="241.3" y="71.12"/>
+<instance part="+3V15" gate="G$1" x="241.3" y="78.74"/>
+<instance part="+3V16" gate="G$1" x="251.46" y="66.04"/>
+<instance part="GND32" gate="1" x="251.46" y="50.8"/>
+<instance part="GND33" gate="1" x="241.3" y="63.5"/>
+<instance part="GND34" gate="1" x="-91.44" y="101.6" rot="R270"/>
 </instances>
 <busses>
@@
 <pinref part="+3V14" gate="G$1" pin="+3V3"/>
 </segment>
+<segment>
+<pinref part="SJ2" gate="G$1" pin="1"/>
+<pinref part="+3V15" gate="G$1" pin="+3V3"/>
+</segment>
+<segment>
+<pinref part="SJ1" gate="G$1" pin="1"/>
+<pinref part="+3V16" gate="G$1" pin="+3V3"/>
+</segment>
 </net>
 <net name="0V" class="0">
@@
 <pinref part="R7" gate="G$1" pin="2"/>
 <pinref part="GND31" gate="1" pin="0V"/>
+</segment>
+<segment>
+<pinref part="SJ1" gate="G$1" pin="3"/>
+<pinref part="GND32" gate="1" pin="0V"/>
+</segment>
+<segment>
+<pinref part="SJ2" gate="G$1" pin="3"/>
+<pinref part="GND33" gate="1" pin="0V"/>
+</segment>
+<segment>
+<pinref part="S1" gate="G$1" pin="1"/>
+<pinref part="GND34" gate="1" pin="0V"/>
 </segment>
 </net>
@@
 <wire x1="-68.58" y1="101.6" x2="-78.74" y2="101.6" width="0.1524" layer="91"/>
 <label x="-76.2" y="101.6" size="1.778" layer="95"/>
+<pinref part="S1" gate="G$1" pin="2"/>
 </segment>
 <segment>
@@
 </segment>
 <segment>
-<wire x1="233.68" y1="91.44" x2="241.3" y2="91.44" width="0.1524" layer="91"/>
 <label x="238.76" y="91.44" size="1.778" layer="95"/>
+<pinref part="U$8" gate="G$1" pin="TXD"/>
+<wire x1="215.9" y1="91.44" x2="241.3" y2="91.44" width="0.1524" layer="91"/>
 </segment>
 </net>
@@
 </segment>
 <segment>
-<wire x1="241.3" y1="93.98" x2="233.68" y2="93.98" width="0.1524" layer="91"/>
-<label x="238.76" y="93.98" size="1.778" layer="95"/>
+<wire x1="236.22" y1="76.2" x2="215.9" y2="76.2" width="0.1524" layer="91"/>
+<label x="226.06" y="76.2" size="1.778" layer="95"/>
+<pinref part="U$8" gate="G$1" pin="EN"/>
 </segment>
 </net>
@@
 </segment>
 </net>
+<net name="N$18" class="0">
+<segment>
+<pinref part="U$8" gate="G$1" pin="P1"/>
+<pinref part="SJ2" gate="G$1" pin="2"/>
+<wire x1="215.9" y1="71.12" x2="236.22" y2="71.12" width="0.1524" layer="91"/>
+</segment>
+</net>
+<net name="N$20" class="0">
+<segment>
+<pinref part="SJ1" gate="G$1" pin="2"/>
+<wire x1="246.38" y1="58.42" x2="226.06" y2="58.42" width="0.1524" layer="91"/>
+<wire x1="226.06" y1="58.42" x2="226.06" y2="66.04" width="0.1524" layer="91"/>
+<pinref part="U$8" gate="G$1" pin="P0"/>
+<wire x1="226.06" y1="66.04" x2="215.9" y2="66.04" width="0.1524" layer="91"/>
+</segment>
+</net>

Commit message: initial route
Parts:
- removed U$9: SARANTEL-SL1250, Ava:SARANTEL-SL1250
- added R10, R8, R9: (no value), rcl:R-EU_R0603
- added SJ3: (no value), jumper:SJ
- added TP1, TP2, TP3: PTR1B2,54, testpad:PTR1B2,54
- added U$5: JDGA-REMQV-ANTENNA, Ava:JDGA-REMQV-ANTENNA
- renumbered U$1 to X3, U$10 to IC4, U$11 to IC3, U$2 to IC1, U$3 to IC2, U$8 to X4
Connections:
- new net N$21: R8.2, SJ3.1, X4.TXD
- net +3V3: now also JP1.VCC, R9.1, TP1.TP
- net 0V: now also R10.2, TP2.TP, U$5.GND; no longer U$9.GND, U$9.GND2
- net N$1: now also U$5.FEED; no longer U$9.FEED
- net N$2: now also TP3.TP
- net TX: now also R10.1, R8.1, R9.2, SJ3.2; no longer X4.TXD
Other:
- note added: "SWDIO is by default pulled high, SWCLK pulled low. LEDs arranged to not be powered by pullups"
- note added: "filter?"

Commit message: routing almost done
Parts:
- removed R10, R8, R9: (no value), rcl:R-EU_R0603
- removed SJ3: (no value), jumper:SJ
- added TP4: PTR1B2,54, testpad:PTR1B2,54
- SV1: device con-lstb:MA03-1 -> Mine:MA03-1
Connections:
- removed net N$21: R8.2, SJ3.1, X4.TXD
- net +3V3: no longer R9.1
- net 0V: no longer R10.2
- net N$6: now also TP4.TP
- net TX: now also X4.TXD; no longer R10.1, R8.1, R9.2, SJ3.2
Changed lines of the file:
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@@
 <part name="R7" library="rcl" deviceset="R-EU_" device="R0603" value="1k"/>
 <part name="+3V14" library="supply1" deviceset="+3V3" device=""/>
-<part name="SV1" library="con-lstb" deviceset="MA03-1" device=""/>
+<part name="SV1" library="Mine" deviceset="MA03-1" device=""/>
 <part name="SJ1" library="jumper" deviceset="SJ2W" device=""/>
 <part name="SJ2" library="jumper" deviceset="SJ2W" device=""/>
@@
 <part name="GND34" library="supply1" deviceset="0V" device=""/>
 <part name="U$5" library="Ava" deviceset="JDGA-REMQV-ANTENNA" device=""/>
-<part name="R8" library="rcl" deviceset="R-EU_" device="R0603"/>
-<part name="R9" library="rcl" deviceset="R-EU_" device="R0603"/>
-<part name="R10" library="rcl" deviceset="R-EU_" device="R0603"/>
-<part name="GND35" library="supply1" deviceset="0V" device=""/>
-<part name="+3V17" library="supply1" deviceset="+3V3" device=""/>
-<part name="SJ3" library="jumper" deviceset="SJ" device=""/>
 <part name="TP1" library="testpad" deviceset="PTR1" device="B2,54"/>
 <part name="TP2" library="testpad" deviceset="PTR1" device="B2,54"/>
 <part name="TP3" library="testpad" deviceset="PTR1" device="B2,54"/>
+<part name="TP4" library="testpad" deviceset="PTR1" device="B2,54"/>
 </parts>
 <sheets>
@@
 <instance part="GND34" gate="1" x="-91.44" y="101.6" rot="R270"/>
 <instance part="U$5" gate="G$1" x="114.3" y="86.36" rot="R180"/>
-<instance part="R8" gate="G$1" x="228.6" y="91.44" rot="R180"/>
-<instance part="R9" gate="G$1" x="233.68" y="104.14" rot="R270"/>
-<instance part="R10" gate="G$1" x="243.84" y="86.36"/>
-<instance part="GND35" gate="1" x="254" y="86.36" rot="R90"/>
-<instance part="+3V17" gate="G$1" x="233.68" y="111.76"/>
-<instance part="SJ3" gate="1" x="223.52" y="96.52"/>
 <instance part="TP1" gate="G$1" x="96.52" y="152.4" rot="R90"/>
 <instance part="TP2" gate="G$1" x="96.52" y="142.24" rot="R90"/>
 <instance part="TP3" gate="G$1" x="27.94" y="119.38" rot="R180"/>
+<instance part="TP4" gate="G$1" x="208.28" y="121.92" rot="R90"/>
 </instances>
 <busses>
@@
 <pinref part="IC4" gate="A" pin="ANT"/>
 <wire x1="193.04" y1="121.92" x2="205.74" y2="121.92" width="0.1524" layer="91"/>
-<wire x1="205.74" y1="121.92" x2="205.74" y2="124.46" width="0.1524" layer="91"/>
+<pinref part="TP4" gate="G$1" pin="TP"/>
 </segment>
 </net>
@@
 </segment>
 <segment>
-<pinref part="R9" gate="G$1" pin="1"/>
-<pinref part="+3V17" gate="G$1" pin="+3V3"/>
-</segment>
-<segment>
 <pinref part="JP1" gate="G$1" pin="VCC"/>
 <pinref part="+3V8" gate="G$1" pin="+3V3"/>
@@
 <pinref part="S1" gate="G$1" pin="1"/>
 <pinref part="GND34" gate="1" pin="0V"/>
-</segment>
-<segment>
-<pinref part="R10" gate="G$1" pin="2"/>
-<pinref part="GND35" gate="1" pin="0V"/>
-<wire x1="251.46" y1="86.36" x2="248.92" y2="86.36" width="0.1524" layer="91"/>
 </segment>
 </net>
@@
 <segment>
 <label x="238.76" y="91.44" size="1.778" layer="95"/>
-<pinref part="R8" gate="G$1" pin="1"/>
-<pinref part="R9" gate="G$1" pin="2"/>
-<wire x1="233.68" y1="91.44" x2="241.3" y2="91.44" width="0.1524" layer="91"/>
-<junction x="233.68" y="91.44"/>
-<pinref part="SJ3" gate="1" pin="2"/>
-<wire x1="228.6" y1="96.52" x2="233.68" y2="96.52" width="0.1524" layer="91"/>
-<wire x1="233.68" y1="96.52" x2="233.68" y2="91.44" width="0.1524" layer="91"/>
-<pinref part="R10" gate="G$1" pin="1"/>
-<wire x1="238.76" y1="86.36" x2="233.68" y2="86.36" width="0.1524" layer="91"/>
-<wire x1="233.68" y1="86.36" x2="233.68" y2="91.44" width="0.1524" layer="91"/>
-<wire x1="233.68" y1="99.06" x2="233.68" y2="96.52" width="0.1524" layer="91"/>
-<junction x="233.68" y="91.44"/>
-<junction x="233.68" y="96.52"/>
-<wire x1="233.68" y1="96.52" x2="233.68" y2="91.44" width="0.1524" layer="91"/>
+<pinref part="X4" gate="G$1" pin="TXD"/>
+<wire x1="215.9" y1="91.44" x2="241.3" y2="91.44" width="0.1524" layer="91"/>
 </segment>
 </net>
@@
 </segment>
 </net>
-<net name="N$21" class="0">
-<segment>
-<pinref part="X4" gate="G$1" pin="TXD"/>
-<pinref part="R8" gate="G$1" pin="2"/>
-<wire x1="215.9" y1="91.44" x2="223.52" y2="91.44" width="0.1524" layer="91"/>
-<pinref part="SJ3" gate="1" pin="1"/>
-<wire x1="218.44" y1="96.52" x2="215.9" y2="96.52" width="0.1524" layer="91"/>
-<wire x1="215.9" y1="96.52" x2="215.9" y2="91.44" width="0.1524" layer="91"/>
-<junction x="215.9" y="91.44"/>
-</segment>
-</net>

Commit message: almost done
Parts:
- removed C13: 1u, rcl:C-EUC0603
- removed TP4: PTR1B2,54, testpad:PTR1B2,54
- removed X4: RADIOMETRIX-MTX2, Ava:RADIOMETRIX-MTX2
- C1, C2, C4: value (none) -> 1u
- C11, C12: value 2u2 -> (none); device rcl:C-EUC0603 -> rcl:C-EUC0805
- C5, C6: value 1u -> (none)
- C7, C8: value (none) -> 2u2; device rcl:C-EUC1210 -> rcl:C-EUC0603
- IC3: value MCP1640 -> RFM69HW; device ukhas:MCP1640 -> hoperf:RFM69HW
- IC4: value RFM69HW -> MCP1640; device hoperf:RFM69HW -> ukhas:MCP1640
- J2: value (none) -> 20-0096; device dtb:JST_2MM_MALE_TH -> ukhas:3.5MMJACKSMD
- R3: value (none) -> 1k
- R7: value 1k -> (none)
- X1: value SMA-142-0701-851/861 -> RADIOMETRIX-MTX2; device con-coax:SMA-142-0701-851/861 -> Ava:RADIOMETRIX-MTX2
- X2: value 1503_02 -> SMA-142-0701-851/861; device con-lumberg:1503_02 -> con-coax:SMA-142-0701-851/861
- renumbered B2 to B1, J1 to J3, U$4 to L1, U$5 to U$2
Connections:
- net +3V3: now also C12.1, C4.2, C5.1, C6.1, IC3.VCC, IC4.VOUT, LED2.A, R4.2, S3.1, X1.VCC; no longer C1.1, C13.2, C2.1, C4.1, C8.1, IC3.VOUT, IC4.VCC, LED1.A, R2.2, S2.1, X4.VCC
- net 0V: now also C11.2, C4.1, C5.2, C6.2, C8.1, IC3.GNDA, IC3.GNDB, IC4.GND, J2.2, LED1.C, R2.1, R3.2, R5.1, S2.1, X1.0V, X1.RFGND; no longer C1.2, C11.1, C13.1, C2.2, C4.2, C8.2, IC3.GND, IC4.GNDA, IC4.GNDB, LED2.C, R3.1, R4.1, R7.2, S1.1, X1.2, X4.0V, X4.RFGND
- net ADC1: now also J2.4; no longer X2.3
- net CS: now also IC3.NSS; no longer IC4.NSS
- net DIO0: now also IC3.DIO0; no longer IC4.DIO0
- net MISO: now also IC3.MISO; no longer IC4.MISO
- net MOSI: now also IC3.MOSI; no longer IC4.MOSI
- net N$10: now also C2.2; no longer C5.2
- net N$11: now also C1.2; no longer C6.2
- net N$12: now also C2.1; no longer C5.1
- net N$13: now also C1.1; no longer C6.1
- net N$14: now also IC4.FB, R4.1, R5.2; no longer IC3.FB, R2.1, R3.2
- net N$15: now also IC4.SW; no longer IC3.SW
- net N$16: now also C7.1; no longer C12.1
- net N$17: now also LED1.A, R7.1; no longer LED2.A, R6.1
- net N$18: now also X1.P1; no longer X4.P1
- net N$19: now also R3.1, S1.1; no longer R7.1, S3.1
- net N$20: now also X1.P0; no longer X4.P0
- net N$3: now also LED2.C, R6.2; no longer LED1.C, R5.2
- net N$4: now also X1.RFOUT, X2.1; no longer X1.1, X4.RFOUT
- net N$5: now also R2.2; no longer R4.2
- net N$6: now also IC3.ANT; no longer IC4.ANT, TP4.TP
- net N$7: now also S3.2; no longer S2.2
- net NRST: now also S2.2; no longer S1.2
- net SCK: now also IC3.SCK; no longer IC4.SCK
- net SWCLK: now also R7.2; no longer R6.2
- net SWDAT: now also R6.1; no longer R5.1
- net TX: now also X1.TXD; no longer X4.TXD
- net TX_EN: now also S1.2, X1.EN; no longer S3.2, X4.EN
- net VCC: now also C8.2; no longer C11.2
- net VIN: now also C11.1, IC4.EN, IC4.VIN; no longer C7.1, IC3.EN, IC3.VIN
Other:
- note added: "2292526"
- note removed: "??"
- moved on the sheet: C1, C10, C11, C12, C2, C3, C4, C5, C6, C7, C8, C9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
